Commit message: update

File: armmp/armmp_description/urdf/armmp_copy.urdf.xacro (robot description, xacro)
@@ -28,8 +28,15 @@
       <dynamics damping="0.7" />
     </joint>
+    <gazebo>
+    <!-- plugin for RobotiQ hand -->
+    <plugin name="robotiq_hand_plugin" filename="libRobotiqHandPlugin.so">
+      <kp_position>10.0</kp_position>
+      <kd_position>0.5</kd_position>
+    </plugin>
+    </gazebo>
     <transmission name="gripper_finger_1_joint_1">
     <type>transmission_interface/SimpleTransmission</type>
     <joint name="gripper_finger_1_joint_1">
-      <hardwareInterface>hardware_interface/EffortJointInterface</hardwareInterface>
+      <hardwareInterface>hardware_interface/PositionJointInterface</hardwareInterface>
     </joint>
     <actuator name="gripper_finger_1_joint_1_motor">
@@ -40,5 +47,5 @@
     <type>transmission_interface/SimpleTransmission</type>
     <joint name="gripper_finger_1_joint_2">
-      <hardwareInterface>hardware_interface/EffortJointInterface</hardwareInterface>
+      <hardwareInterface>hardware_interface/PositionJointInterface</hardwareInterface>
     </joint>
     <actuator name="gripper_finger_1_joint_2_motor">
@@ -49,5 +56,5 @@
     <type>transmission_interface/SimpleTransmission</type>
     <joint name="gripper_finger_1_joint_3">
-      <hardwareInterface>hardware_interface/EffortJointInterface</hardwareInterface>
+      <hardwareInterface>hardware_interface/PositionJointInterface</hardwareInterface>
     </joint>
     <actuator name="gripper_finger_1_joint_3_motor">
@@ -58,5 +65,5 @@
     <type>transmission_interface/SimpleTransmission</type>
     <joint name="gripper_finger_2_joint_1">
-      <hardwareInterface>hardware_interface/EffortJointInterface</hardwareInterface>
+      <hardwareInterface>hardware_interface/PositionJointInterface</hardwareInterface>
     </joint>
     <actuator name="gripper_finger_2_joint_1_motor">
@@ -67,5 +74,5 @@
     <type>transmission_interface/SimpleTransmission</type>
     <joint name="gripper_finger_2_joint_2">
-      <hardwareInterface>hardware_interface/EffortJointInterface</hardwareInterface>
+      <hardwareInterface>hardware_interface/PositionJointInterface</hardwareInterface>
     </joint>
     <actuator name="gripper_finger_2_joint_2_motor">
@@ -76,5 +83,5 @@
     <type>transmission_interface/SimpleTransmission</type>
     <joint name="gripper_finger_2_joint_3">
-      <hardwareInterface>hardware_interface/EffortJointInterface</hardwareInterface>
+      <hardwareInterface>hardware_interface/PositionJointInterface</hardwareInterface>
     </joint>
     <actuator name="gripper_finger_2_joint_3_motor">
@@ -85,5 +92,5 @@
     <type>transmission_interface/SimpleTransmission</type>
     <joint name="gripper_finger_middle_joint_1">
-      <hardwareInterface>hardware_interface/EffortJointInterface</hardwareInterface>
+      <hardwareInterface>hardware_interface/PositionJointInterface</hardwareInterface>
     </joint>
     <actuator name="gripper_finger_middle_joint_1_motor">
@@ -94,5 +101,5 @@
     <type>transmission_interface/SimpleTransmission</type>
     <joint name="gripper_finger_middle_joint_2">
-      <hardwareInterface>hardware_interface/EffortJointInterface</hardwareInterface>
+      <hardwareInterface>hardware_interface/PositionJointInterface</hardwareInterface>
     </joint>
     <actuator name="gripper_finger_middle_joint_2_motor">
@@ -103,5 +110,5 @@
     <type>transmission_interface/SimpleTransmission</type>
     <joint name="gripper_finger_middle_joint_3">
-      <hardwareInterface>hardware_interface/EffortJointInterface</hardwareInterface>
+      <hardwareInterface>hardware_interface/PositionJointInterface</hardwareInterface>
     </joint>
     <actuator name="gripper_finger_middle_joint_3">
@@ -112,5 +119,5 @@
     <type>transmission_interface/SimpleTransmission</type>
     <joint name="gripper_palm_finger_1_joint">
-      <hardwareInterface>hardware_interface/EffortJointInterface</hardwareInterface>
+      <hardwareInterface>hardware_interface/PositionJointInterface</hardwareInterface>
     </joint>
     <actuator name="gripper_palm_finger_1_joint_motor">
@@ -121,5 +128,5 @@
     <type>transmission_interface/SimpleTransmission</type>
     <joint name="gripper_palm_finger_2_joint">
-      <hardwareInterface>hardware_interface/EffortJointInterface</hardwareInterface>
+      <hardwareInterface>hardware_interface/PositionJointInterface</hardwareInterface>
     </joint>
     <actuator name="gripper_palm_finger_1_joint_motor">
@@ -280,8 +287,8 @@
 		</arm>
 	       <forces_angle_tolerance>100</forces_angle_tolerance>
-	       <update_rate>4</update_rate>
-	       <grip_count_threshold>4</grip_count_threshold>
-	       <max_grip_count>8</max_grip_count>
-	       <release_tolerance>0.005</release_tolerance>
+	       <update_rate>20</update_rate>
+	       <grip_count_threshold>1</grip_count_threshold>
+	       <max_grip_count>3</max_grip_count>
+	       <release_tolerance>0.0198</release_tolerance>
 	       <disable_collisions_on_attach>false</disable_collisions_on_attach>
 	       <contact_topic>__default_topic__</contact_topic>
@@ -291,8 +298,33 @@
 <xacro:ur10e_robotiq prefix=""/>
   <link name="world" />
-  <joint name="world_joint" type="fixed">
-    <parent link="world" />
+    <!-- Stand -->
+  <link name="stand">
+    <inertial>
+        <mass value="1000" />
+        <origin xyz="0 0 0.5" rpy="0 0 0" />
+        <inertia ixx="0.01" ixy="0" ixz="0" iyy="0.01" iyz="0" izz="0.01" />
+    </inertial>
+    <visual>
+        <origin xyz="0 0 0.5" rpy="0 0 0" />
+        <geometry>
+            <cylinder length="1.0" radius="0.1" />
+        </geometry>
+    </visual>
+    <collision>
+        <origin xyz="0 0 0.5" rpy="0 0 0" />
+        <geometry>
+            <!-- <box size="0.2 0.2 1.0" /> -->
+            <cylinder length="1.0" radius="0.1" />
+        </geometry>
+    </collision>
+  </link>
+  <joint name="fixed" type="fixed">
+    <parent link="world"/>
+    <child link="stand"/>
+  </joint>
+  <joint name="stand_joint" type="fixed">
+    <parent link="stand" />
     <child link = "base_link" />
-    <origin xyz="0.0 0.0 0.0" rpy="0.0 0.0 0.0" />
+    <origin xyz="0.0 0.0 1.0" rpy="0.0 0.0 0.0" />
   </joint>
 </robot>
